File: kicad/LoRa-Phone.kicad_pcb (KiCad board)
At the start: 4 copper layers, 50 x 86 mm, 78 parts, among them IC1 E22-900M22S, IC2 ESP32-S3-MINI-1-N8, IC3 TPS62842DGRR, IC4 MCP23017-E_SO, IC5 L86-M33, J1 USB_C, J2 WS2812B, J3 Conn_02x07_Top_Bottom, J4 Conn_Coaxial, M1 Motor_DC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

Commit message: Third version
Parts:
- added C19: 1uF, Capacitor_SMD:C_0603_1608Metric, B.Cu at (190.6, 63.7)
- added C20: 1uF, Capacitor_SMD:C_0603_1608Metric, B.Cu at (188.7, 66.2)
- added J5: LED0, Connector_PinHeader_1.27mm:PinHeader_2x02_P1.27mm_Vertical, B.Cu at (190.5, 51.5)
- added J6: LED1, Connector_PinHeader_1.27mm:PinHeader_2x02_P1.27mm_Vertical, B.Cu at (197.0, 50.3)
- added J7: LED2, Connector_PinHeader_1.27mm:PinHeader_2x02_P1.27mm_Vertical, B.Cu at (190.5, 55.9)
- added J8: LED3, Connector_PinHeader_1.27mm:PinHeader_2x02_P1.27mm_Vertical, B.Cu at (197.0, 54.7)
- added J9: ROTARY_ENCODER, Connector_PinHeader_1.27mm:PinHeader_1x03_P1.27mm_Vertical, F.Cu at (166.2, 49.8)
- added R28: 5K, Resistor_SMD:R_0603_1608Metric, B.Cu at (194.8, 73.2)
- added R29: 10K, Resistor_SMD:R_0603_1608Metric, F.Cu at (162.9, 109.0)
- added R30: 10K, Resistor_SMD:R_0603_1608Metric, F.Cu at (166.1, 110.7)
- added U4: PLP5012PWR, LoRa-Phone:TSSOP24_PW_TEX, B.Cu at (195.4, 66.8)
- added U5: MAX16150AUT+T, LoRa-Phone:21-0058I_MXM, F.Cu at (164.4, 120.0)
- J1: footprint Connector_PinHeader_2.54mm:PinHeader_1x04_P2.54mm_Vertical -> Connector_PinHeader_1.27mm:PinHeader_1x04_P1.27mm_Vertical
- J2: value WS2812B -> BUTTON; footprint Connector_PinHeader_1.27mm:PinHeader_1x03_P1.27mm_Vertical -> Connector_PinHeader_1.27mm:PinHeader_1x02_P1.27mm_Vertical
- SW1: value Power_Switch -> SW_Push
- moved J2 46.7 mm to (163.7, 54.5)
- moved G*** 32.5 mm to (193.8, 52.9)
- moved SW1 23.4 mm to (164.6, 124.2), turned to -90 degrees
- moved R11 15.3 mm to (177.3, 51.2)
- moved Q1 12.0 mm to (185.4, 52.1), turned to -90 degrees
- moved R10 11.7 mm to (180.9, 51.2), turned to 0 degrees
- moved R26 1.22 mm to (168.1, 116.2)
- moved R25 1.22 mm to (170.4, 118.6)
Connections:
- C13 pad 1: VCC -> VCC_AS
- C2 pad 2: VCC -> VCC_AS
- IC2 pad 14: CUST_GPIO1 -> INT_POWER
- IC2 pad 15: CUST_GPIO2 -> CLR_POWER
- IC2 pad 30: LED_DATA -> CUST_GPIO6
- IC2 pad 9: MCP_INTB -> BUTTON
- IC3 pad 5: VCC_AS -> EN_POWER
- IC4 pad 19: MCP_INTB -> unconnected-(IC4-INTB-Pad19)
- J2 pad 1: +3V3 -> GND
- J2 pad 2: LED_DATA -> BUTTON
- J3 pad 12: GPA2 -> CUST_GPIO6
- J3 pad 8: CUST_GPIO1 -> GND
- J3 pad 9: CUST_GPIO2 -> GND
- SW1 pad 1: VCC -> GND
- SW1 pad 2: VCC_AS -> Net-(U5-*PB_IN)
- U2 pad 10: VCC -> VCC_AS
- U2 pad 11: VCC -> VCC_AS
Routing:
- net MCP_INTB: track 109.1 -> 0.00 mm, vias 2 -> 0
- net BUTTON: track 0.00 -> 102.7 mm, vias 0 -> 3
- net CUST_GPIO1: track 85.4 -> 0.00 mm, vias 9 -> 0
- net INT_POWER: track 0.00 -> 84.5 mm, vias 0 -> 6
- net CLR_POWER: track 0.00 -> 84.3 mm, vias 0 -> 6
- net CUST_GPIO6: track 0.00 -> 75.2 mm, vias 0 -> 4
- net CUST_GPIO2: track 71.6 -> 0.00 mm, vias 6 -> 0
- net SCL: track 153.4 -> 204.6 mm, vias 10 -> 13
- net SDA: track 145.5 -> 196.3 mm, vias 10 -> 13
- net Net-(J5-Pin_3): track 0.00 -> 28.6 mm
- net Net-(J5-Pin_2): track 0.00 -> 23.2 mm
- net Net-(J5-Pin_1): track 0.00 -> 22.9 mm
- net Net-(J6-Pin_3): track 0.00 -> 22.4 mm
- net Net-(J6-Pin_1): track 0.00 -> 21.7 mm
- net Net-(J6-Pin_2): track 0.00 -> 19.9 mm
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- added copper zone on B.Cu, net VCC_AS
- added copper zone on F.Cu, net VCC_AS
- removed copper zone on B.Cu, net VCC
- removed copper zone on F.Cu, net VCC
