File: kicad/LoRa-Phone.kicad_sch (KiCad schematic)
At the start: 73 parts, among them IC1 E22-900M22S, IC2 ESP32-S3-MINI-1-N8, IC3 TPS62842DGRR, IC4 MCP23017-E_SO, IC5 L86-M33, J1 USB_C, J2 WS2812B, J3 Conn_02x07_Top_Bottom, J4 Conn_Coaxial, M1 Motor_DC, Q1 AO3400A, Q2 AO3401A, SW1 Power_Switch, SW2 BOOT, SW3 RESET, U1 MAX98357A, U2 BQ24072RGT, U3 MAX17048G_T10

Commit message: Third version
Parts:
- removed J2: WS2812B, Connector_PinHeader_1.27mm:PinHeader_1x03_P1.27mm_Vertical, symbol Connector:Conn_01x03_Socket
- removed SW1: Power_Switch, Connector_PinHeader_1.27mm:PinHeader_1x02_P1.27mm_Vertical, symbol Switch:SW_DIP_x01
- added C19, C20: 1uF, Capacitor_SMD:C_0603_1608Metric, symbol Device:C_Small
- added J2: BUTTON, Connector_PinHeader_1.27mm:PinHeader_1x02_P1.27mm_Vertical, symbol Connector:Conn_01x02_Socket
- added J5: LED0, Connector_PinHeader_1.27mm:PinHeader_2x02_P1.27mm_Vertical, symbol Connector:Conn_01x04_Socket
- added J6: LED1, Connector_PinHeader_1.27mm:PinHeader_2x02_P1.27mm_Vertical, symbol Connector:Conn_01x04_Socket
- added J7: LED2, Connector_PinHeader_1.27mm:PinHeader_2x02_P1.27mm_Vertical, symbol Connector:Conn_01x04_Socket
- added J8: LED3, Connector_PinHeader_1.27mm:PinHeader_2x02_P1.27mm_Vertical, symbol Connector:Conn_01x04_Socket
- added J9: ROTARY_ENCODER, Connector_PinHeader_1.27mm:PinHeader_1x03_P1.27mm_Vertical, symbol Connector:Conn_01x03_Socket
- added R28: 5K, Resistor_SMD:R_0603_1608Metric, symbol Device:R_Small_US
- added R29, R30: 10K, Resistor_SMD:R_0603_1608Metric, symbol Device:R_Small_US
- added SW1: SW_Push, Connector_PinHeader_1.27mm:PinHeader_1x02_P1.27mm_Vertical, symbol Switch:SW_Push
- added U4: PLP5012PWR, LoRa-Phone:TSSOP24_PW_TEX, symbol LoRa-Phone:PLP5012PWR
- added U5: MAX16150AUT+T, LoRa-Phone:21-0058I_MXM, symbol LoRa-Phone:MAX16150AUT+T
- J1: footprint Connector_PinHeader_2.54mm:PinHeader_1x04_P2.54mm_Vertical -> Connector_PinHeader_1.27mm:PinHeader_1x04_P1.27mm_Vertical
Connections:
- net +3V3: now also R29.1, R30.1
- net +3V3_NSY: now also C20.1, U4.4 (VCC), U4.8 (EN)
- net GND: now also J3.8 (Pin_8), J3.9 (Pin_9), C19.2, C20.2, J2.1 (Pin_1), J5.4 (Pin_4), J6.4 (Pin_4), J7.4 (Pin_4), J8.4 (Pin_4), J9.3 (Pin_3), R28.2, SW1.1, U4.1 (ADDR0), U4.18 (DGND), U4.2 (AGND), U4.3 (ADDR1), U4.6 (PGND), U5.2 (GND)
- net GPA1: now also J9.1 (Pin_1)
- net GPA2: now also J9.2 (Pin_2); no longer J3.12 (Pin_12)
- net SCL: now also U4.7 (SCL)
- net SDA: now also U4.5 (SDA)
- net VCC: now also C3.2, IC3.6 (VIN), J3.13 (Pin_13), R25.1, U5.3 (VCC)
- net CUST_GPIO1 renamed INT_POWER
- net INT_POWER: now also R30.2, U5.5 (*INT); no longer J3.8 (Pin_8)
- net CUST_GPIO2 renamed CLR_POWER
- net CLR_POWER: now also R29.2, U5.6 (*CLR); no longer J3.9 (Pin_9)
- net LED_DATA renamed CUST_GPIO6
- net CUST_GPIO6: now also J3.12 (Pin_12)
- net MCP_INTB: no longer names the net of IC4.19 (INTB)
- net MCP_INTB: no longer IC2.9 (IO5)
- removed net VCC_AS: C3.2, IC3.5 (EN), IC3.6 (VIN), J3.13 (Pin_13), R25.1
- new net: J7.1 (Pin_1), U4.17 (OUT5)
- new net: J7.2 (Pin_2), U4.16 (OUT4)
- new net: J7.3 (Pin_3), U4.15 (OUT3)
- new net: J6.1 (Pin_1), U4.21 (OUT8)
- new net: J6.2 (Pin_2), U4.20 (OUT7)
- new net: J6.3 (Pin_3), U4.19 (OUT6)
- new net: SW1.2, U5.1 (*PB_IN)
- new net: C19.1, U4.10 (VCAP)
- new net: J8.3 (Pin_3), U4.12 (OUT0)
- new net: J8.2 (Pin_2), U4.13 (OUT1)
- new net: J8.1 (Pin_1), U4.14 (OUT2)
- new net: J5.3 (Pin_3), U4.22 (OUT9)
- new net: J5.2 (Pin_2), U4.23 (OUT10)
- new net: J5.1 (Pin_1), U4.24 (OUT11)
- new net: R28.1, U4.9 (IREF)
- new net BUTTON: IC2.9 (IO5), J2.2 (Pin_2)
- new net EN_POWER: IC3.5 (EN), U5.4 (OUT)
- no-connect marks 5 -> 6
Other:
- note added: "LEDS"
- moved on the sheet: 2.8_TFT_SPI1, AE1, BT1, C1, C10, C11, C12, C13, C14, C15, C16, C17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
